Commit message: Just need to tune PID now.

File: src/en613_description/urdf/basic_robot.gazebo.xacro (robot description, xacro)
@@ -9,5 +9,5 @@
         <topic>/cmd_vel</topic>
         <odom_topic>/odom</odom_topic>
-        <tf_topic>/tf</tf_topic>
+        <tf_topic>/basic_robot/tf</tf_topic>
         <wheel_separation>0.825</wheel_separation>
         <wheel_radius>0.4</wheel_radius>
@@ -28,9 +28,11 @@
         filename="gz-sim-pose-publisher-system"
         name="gz::sim::systems::PosePublisher">
+        <publish_model_pose>true</publish_model_pose>
         <publish_link_pose>true</publish_link_pose>
+        <publish_nested_model_pose>true</publish_nested_model_pose>
         <use_pose_vector_msg>true</use_pose_vector_msg>
-        <update_frequency>-1</update_frequency>
+        <update_frequency>30</update_frequency>
         <static_publisher>true</static_publisher>
-        <static_update_frequency>-1</static_update_frequency>
+        <static_update_frequency>30</static_update_frequency>
       </plugin>
     </gazebo>

File: src/en613_description/urdf/basic_robot_macro.urdf.xacro (robot description, xacro)
@@ -120,5 +120,5 @@
             <inertial>
                 <origin xyz="0 0 0" rpy="0 0 0"/>
-                <mass value="0.1"/>
+                <mass value="0.01"/>
                 <inertia ixx="3.90625e-05" ixy="0.0" ixz="0.0" iyy="3.90625e-05" iyz="0.0" izz="3.90625e-05" />
             </inertial>

Commit message: Ready to turn in!

File: src/en613_description/urdf/basic_robot.gazebo.xacro (robot description, xacro)
@@ -12,11 +12,9 @@
         <wheel_separation>0.825</wheel_separation>
         <wheel_radius>0.4</wheel_radius>
-        <odom_publish_frequency>15</odom_publish_frequency>
+        <odom_publish_frequency>50</odom_publish_frequency>
         <frame_id>odom</frame_id>
         <child_frame_id>chassis</child_frame_id>
-        <max_linear_velocity>0.5</max_linear_velocity>
-        <min_linear_velocity>-0.5</min_linear_velocity>
-        <max_angular_velocity>3.14159</max_angular_velocity>
-        <min_angular_velocity>-3.14159</min_angular_velocity>
+        <max_linear_velocity>2.0</max_linear_velocity>
+        <max_angular_velocity>6.28</max_angular_velocity>
       </plugin>
       <plugin

File: src/en613_description/urdf/basic_robot_macro.urdf.xacro (robot description, xacro)
@@ -24,5 +24,5 @@
             </visual>
             <inertial>
-                <origin xyz="0 0 0" rpy="0 0 0"/>
+                <origin xyz="0 0 -0.25" rpy="0 0 0"/>
                 <mass value="15.0"/>
                 <inertia ixx="0.8578125" ixy="0.0" ixz="0.0" iyy="0.8578125" iyz="0.0" izz="1.7015625" />
@@ -35,14 +35,8 @@
                     <friction>
                         <ode>
-                            <mu>0.5</mu>
-                            <mu2>0.5</mu2>
+                            <mu>0.8</mu>
+                            <mu2>0.8</mu2>
                         </ode>
                     </friction>
-                    <contact>
-                        <ode>
-                            <kp>1e6</kp>
-                            <kd>100</kd>
-                        </ode>
-                    </contact>
                 </surface>
             </collision>
@@ -69,9 +63,6 @@
                     <friction>
                         <ode>
-                            <mu>1</mu>
-                            <mu2>1</mu2>
-                            <slip1>0.035</slip1>
-                            <slip2>0</slip2>
-                            <fdir1>0 0 1</fdir1>
+                            <mu>1.2</mu>
+                            <mu2>1.2</mu2>
                         </ode>
                     </friction>
@@ -100,9 +91,6 @@
                     <friction>
                         <ode>
-                            <mu>1</mu>
-                            <mu2>1</mu2>
-                            <slip1>0.035</slip1>
-                            <slip2>0</slip2>
-                            <fdir1>0 0 1</fdir1>
+                            <mu>1.2</mu>
+                            <mu2>1.2</mu2>
                         </ode>
                     </friction>
@@ -120,6 +108,12 @@
             <inertial>
                 <origin xyz="0 0 0" rpy="0 0 0"/>
-                <mass value="0.01"/>
-                <inertia ixx="3.90625e-05" ixy="0.0" ixz="0.0" iyy="3.90625e-05" iyz="0.0" izz="3.90625e-05" />
+                <mass value="0.002"/>
+                <inertia
+                    ixx="7.8125e-07"
+                    ixy="0.0"
+                    ixz="0.0"
+                    iyy="7.8125e-07"
+                    iyz="0.0"
+                    izz="7.8125e-07"/>
             </inertial>
             <collision>
@@ -134,6 +128,6 @@
             <child link="left_wheel"/>
             <axis xyz="0 1 0"/>
-            <limit effort="100" velocity="10.0"/>
-            <dynamics damping="0.1" friction="0.1"/>
+            <limit effort="100" velocity="5.0"/>
+            <dynamics damping="0.5" friction="0.2"/>
         </joint>
         <joint name="right_wheel_joint" type="continuous">
@@ -142,6 +136,6 @@
             <child link="right_wheel"/>
             <axis xyz="0 1 0"/>
-            <limit effort="100" velocity="10.0"/>
-            <dynamics damping="0.1" friction="0.1"/>
+            <limit effort="100" velocity="5.0"/>
+            <dynamics damping="0.5" friction="0.2"/>
         </joint>
         <joint name="lidar_joint" type="fixed">
